Commit message: Fix Xacro Description

File: yumi_description/urdf/yumi.urdf.xacro (robot description, xacro)
@@ -11,4 +11,8 @@
   <!-- Import Gazebo plugins -->
   <xacro:include filename="$(find yumi_description)/urdf/Gazebo/gazebo.urdf.xacro"/>
+  <xacro:arg name="arms_interface" default="VelocityJointInterface"/>
+  <xacro:arg name="grippers_interface" default="EffortJointInterface"/>
+  <xacro:arg name="yumi_setup" default="robot_centric"/>
+  <xacro:property name="yumi_setup" value="$(arg yumi_setup)" />
   <!--yumi-->
   <xacro:yumi name="yumi" hardware_interface="hardware_interface/$(arg arms_interface)" parent="${yumi_parent}" >
@@ -27,12 +31,10 @@
   	<!-- Pure YuMi URDF, with no joints connecting it to any other robot or pedestal. Neither accessories. -->
   </xacro:if>
-  <xacro:if value="${yumi_setup == 'default'}">
-    <xacro:property name="yumi_parent" value="world" />
-    <link name="world"/>
-    <joint name="world_joint" type="fixed">
-      <parent link="world"/>
-      <child link="yumi_base_link"/>
-      <origin xyz="0 0 0.1" rpy="0 0 0" />
-    </joint>
-  </xacro:if>
+  <xacro:property name="yumi_parent" value="world" />
+  <link name="world"/>
+  <joint name="world_joint" type="fixed">
+    <parent link="world"/>
+    <child link="yumi_base_link"/>
+    <origin xyz="0 0 0.1" rpy="0 0 0" />
+  </joint>
 </robot>

Commit message: Fix Xacro URDF

File: yumi_description/urdf/yumi.urdf.xacro (robot description, xacro)
@@ -14,4 +14,5 @@
   <xacro:arg name="grippers_interface" default="EffortJointInterface"/>
   <xacro:arg name="yumi_setup" default="robot_centric"/>
+  <xacro:arg name="yumi_parent" default="world"/>
   <xacro:property name="yumi_setup" value="$(arg yumi_setup)" />
   <!--yumi-->
@@ -27,5 +28,4 @@
     <origin xyz="0 0 0.007" rpy="0 0 ${PI}" />
   </xacro:yumi_servo_gripper>
-  <xacro:property name="yumi_setup" value="$(arg yumi_setup)" />
   <xacro:if value="${yumi_setup == 'robot_centric'}">
   	<!-- Pure YuMi URDF, with no joints connecting it to any other robot or pedestal. Neither accessories. -->
